Commit message: Forgot to add in xacro variables, fixed

File: nuturtle_description/urdf/turtlebot3_burger.urdf.xacro (robot description, xacro)
@@ -76,5 +76,5 @@
     <parent link="base_link"/>
     <child link="wheel_left_link"/>
-    <origin xyz="0.0 0.08 0.023" rpy="-1.57 0 0"/>
+    <origin xyz="0.0 ${track_width} 0.023" rpy="-1.57 0 0"/>
     <axis xyz="0 0 1"/>
   </joint>
@@ -90,5 +90,5 @@
       <origin xyz="0 0 0" rpy="0 0 0"/>
       <geometry>
-        <cylinder length="0.018" radius="0.033"/>
+        <cylinder length="0.018" radius="${wheel_radius}"/>
       </geometry>
     </collision>
@@ -102,5 +102,5 @@
     <parent link="base_link"/>
     <child link="wheel_right_link"/>
-    <origin xyz="0.0 -0.080 0.023" rpy="-1.57 0 0"/>
+    <origin xyz="0.0 -${track_width/2} 0.023" rpy="-1.57 0 0"/>
     <axis xyz="0 0 1"/>
   </joint>
@@ -116,5 +116,5 @@
       <origin xyz="0 0 0" rpy="0 0 0"/>
       <geometry>
-        <cylinder length="0.018" radius="0.033"/>
+        <cylinder length="0.018" radius="${wheel_radius}"/>
       </geometry>
     </collision>

Commit message: The launch file works and step A.4 is complete
AFter much troubleshooting, the launchfile works and everything is
loaded in correctly with the correct prefixes and everyitng. now I must
go around and add separate rviz files for each color and add logic to
the launch file for using them.

File: nuturtle_description/urdf/turtlebot3_burger.urdf.xacro (robot description, xacro)
@@ -3,12 +3,13 @@
   xmlns:xacro="http://ros.org/wiki/xacro">
   <!-- <xacro:include filename="$(find nuturtle_description)/urdf/common_properties.urdf"/> -->
-<xacro:property name="yaml_file" value="$(find nuturtle_description)/diff_params.yaml"/>
-<xacro:property name="params" value="${xacro.load_yaml(yaml_file)['/**']['ros__parameters']}"/>
-<xacro:property name="wheel_radius" value="${params['wheel_radius']}"/>
-<xacro:property name="track_width" value="${params['track_width']}"/>
-<xacro:property name="motor_cmd_max" value="${params['motor_cmd_max']}"/>
-<xacro:property name="motor_cmd_per_rad_sec" value="${params['motor_cmd_per_rad_sec']}"/>
-<xacro:property name="encoder_ticks_per_rad" value="${params['encoder_ticks_per_rad']}"/>
-<xacro:property name="collision_radius" value="${params['collision_radius']}"/>
+  <xacro:property name="yaml_file" value="$(find nuturtle_description)/config/diff_params.yaml"/>
+  <xacro:property name="params" value="${xacro.load_yaml(yaml_file)['/**']['ros__parameters']}"/>
+  <xacro:property name="wheel_radius" value="${params['wheel_radius']}"/>
+  <xacro:property name="track_width" value="${params['track_width']}"/>
+  <xacro:property name="motor_cmd_max" value="${params['motor_cmd_max']}"/>
+  <xacro:property name="motor_cmd_per_rad_sec" value="${params['motor_cmd_per_rad_sec']}"/>
+  <xacro:property name="encoder_ticks_per_rad" value="${params['encoder_ticks_per_rad']}"/>
+  <xacro:property name="collision_radius" value="${params['collision_radius']}"/>
+  <xacro:arg name="color" default="purple"/>
   <!-- Init colour -->
   <material name="black">
@@ -42,4 +43,7 @@
     <color rgba="1.0 1.0 1.0 1.0"/>
   </material>
+  <material name="purple">
+    <color rgba="0.3 0.16 0.52 1.0"/>
+  </material>
   <link name="base_footprint"/>
   <joint name="base_joint" type="fixed">
@@ -52,12 +56,23 @@
       <origin xyz="-0.032 0 0.0" rpy="0 0 0"/>
       <geometry>
-        <mesh filename="package://nuturtle_description/meshes/bases/burger_base.stl" scale="0.001 0.001 0.001"/>
+        <mesh filename="package://nuturtle_description/meshes/burger_base.stl" scale="0.001 0.001 0.001"/>
       </geometry>
-      <material name="light_black"/>
+      <xacro:if value = "${'color' == 'red'}">
+        <material name="red"/>
+      </xacro:if>
+      <xacro:if value = "${'color' == 'green'}">
+        <material name="green"/>
+      </xacro:if>
+      <xacro:if value = "${'color' == 'blue'}">
+        <material name="blue"/>
+      </xacro:if>
+      <xacro:if value = "${'color' == 'purple'}">
+        <material name="purple"/>
+      </xacro:if>
     </visual>
     <collision>
       <origin xyz="-0.032 0 0.070" rpy="0 0 0"/>
       <geometry>
-        <xacro:if value="${collision_radius} < 0">
+        <xacro:if value="${collision_radius == 0}">
           <box size="0.140 0.140 0.143"/>
         </xacro:if>
@@ -76,5 +91,5 @@
     <parent link="base_link"/>
     <child link="wheel_left_link"/>
-    <origin xyz="0.0 ${track_width} 0.023" rpy="-1.57 0 0"/>
+    <origin xyz="0.0 ${track_width/2} 0.023" rpy="-1.57 0 0"/>
     <axis xyz="0 0 1"/>
   </joint>
@@ -83,5 +98,5 @@
       <origin xyz="0 0 0" rpy="1.57 0 0"/>
       <geometry>
-        <mesh filename="package://nuturtle_description/meshes/wheels/left_tire.stl" scale="0.001 0.001 0.001"/>
+        <mesh filename="package://nuturtle_description/meshes/left_tire.stl" scale="0.001 0.001 0.001"/>
       </geometry>
       <material name="dark"/>
@@ -109,5 +124,5 @@
       <origin xyz="0 0 0" rpy="1.57 0 0"/>
       <geometry>
-        <mesh filename="package://nuturtle_description/meshes/wheels/right_tire.stl" scale="0.001 0.001 0.001"/>
+        <mesh filename="package://nuturtle_description/meshes/right_tire.stl" scale="0.001 0.001 0.001"/>
       </geometry>
       <material name="dark"/>
@@ -158,5 +173,5 @@
       <origin xyz="0 0 0.0" rpy="0 0 0"/>
       <geometry>
-        <mesh filename="package://nuturtle_description/meshes/sensors/lds.stl" scale="0.001 0.001 0.001"/>
+        <mesh filename="package://nuturtle_description/meshes/lds.stl" scale="0.001 0.001 0.001"/>
       </geometry>
       <material name="dark"/>

Commit message: Finished task A.4
Added in the capability to create a turtlebot of any of the predefined
colors just with a launch file arguement. Everything seems to be working
fine.

File: nuturtle_description/urdf/turtlebot3_burger.urdf.xacro (robot description, xacro)
@@ -12,4 +12,5 @@
   <xacro:property name="collision_radius" value="${params['collision_radius']}"/>
   <xacro:arg name="color" default="purple"/>
+  <xacro:property name="color" value="$(arg color)"/>
   <!-- Init colour -->
   <material name="black">
@@ -58,15 +59,15 @@
         <mesh filename="package://nuturtle_description/meshes/burger_base.stl" scale="0.001 0.001 0.001"/>
       </geometry>
-      <xacro:if value = "${'color' == 'red'}">
-        <material name="red"/>
+      <xacro:if value="${color == 'blue'}">
+        <material name="${color}"/>
       </xacro:if>
-      <xacro:if value = "${'color' == 'green'}">
-        <material name="green"/>
+      <xacro:if value = "${color == 'green'}">
+        <material name="${color}"/>
       </xacro:if>
-      <xacro:if value = "${'color' == 'blue'}">
-        <material name="blue"/>
+      <xacro:if value = "${color == 'blue'}">
+        <material name="${color}"/>
       </xacro:if>
-      <xacro:if value = "${'color' == 'purple'}">
-        <material name="purple"/>
+      <xacro:if value = "${color == 'purple'}">
+        <material name="${color}"/>
       </xacro:if>
     </visual>
